File: HaptiCare design.kicad_sch (KiCad schematic)
At the start: 51 parts, among them IC1 IP5306, J1 Conn_01x02_Socket, J2 Conn_01x02_Socket, J3 Conn_01x02_Socket, J4 Conn_01x02_Socket, J5 USB_C_Receptacle, J6 oled, Q1 AO3400A, Q2 AO3400A, Q3 AO3400A, Q4 AO3400A, SW1 SW_Push, U1 ESP32-S3-WROOM-1, U2 ME6211C33M5

Commit message: Update power management, ESP32 programming, and sub-schematics
Parts:
- added C12: 22uF, symbol Device:C
- added C13: 0.1uF, symbol Device:C
- added C14: 1uF, symbol Device:C
- added J7: Conn_01x04_Pin, symbol Connector:Conn_01x04_Pin
- added J8: Battery, symbol Connector_Generic:Conn_01x02
- added R15: 10k, symbol Device:R_US
- added SW2, SW3: SW_Push, symbol Switch:SW_Push
- L1: value L -> 1uH
Connections:
- net GND: now also C12.2, C13.2, C14.1, J7.1 (Pin_1), J8.2 (Pin_2), SW2.1, SW3.1
- net vout2: now also C12.1, C13.1, J7.4 (Pin_4), R15.2
- net USB D+: now reaches J5.A6 (D+)
- net USB D+: now also J5.B6 (D+), U1.14 (USB_D+)
- net USB D-: now reaches J5.A7 (D-)
- net USB D-: now also J5.B7 (D-), U1.13 (USB_D-)
- net BAT: now reaches C6.1, IC1.6 (BAT), L1.2, R1.1
- net BAT: now also J8.1 (Pin_1)
- net at U1.27 (IO0): now also SW3.2
- net at U1.3 (EN): now also C14.2, R15.1, SW2.2
- net RXD0: now reaches U1.36 (RXD0)
- net RXD0: now also J7.2 (Pin_2)
- net TXD0: now reaches U1.37 (TXD0)
- net TXD0: now also J7.3 (Pin_3)
- no-connect marks 1 -> 4
Other:
- moved on the sheet: U1

Commit message: Add ESD protection and change net names
Parts:
- removed J7: Conn_01x04_Pin, symbol Connector:Conn_01x04_Pin
- removed J8: Battery, symbol Connector_Generic:Conn_01x02
- added C15: NC, symbol Device:C
- added D10, D11: SP3530-01ETG, symbol Device:D_TVS
- added D12: SMBJ58A, symbol Device:D_TVS
- added J10, J7: Conn_01x03, symbol Connector_Generic:Conn_01x03
- added J9: Conn_01x06_Pin, symbol Connector:Conn_01x06_Pin
- added R16: 0, symbol Device:R
Connections:
- net BAT: now also J7.1 (Pin_1), J7.2 (Pin_2), J7.3 (Pin_3), R16.1; no longer IC1.6 (BAT)
- net GND: now also C15.2, D10.1 (A1), D11.1 (A1), D12.1 (A1), J10.1 (Pin_1), J10.2 (Pin_2), J10.3 (Pin_3), J9.1 (Pin_1)
- net RXD0: now also J9.4 (Pin_4)
- net TXD0: now also J9.5 (Pin_5)
- net USB D+: now also D10.2 (A2)
- net USB D-: now also D11.2 (A2)
- net Vbus: now also D12.2 (A2)
- net Reset: now reaches C14.2, R15.1, SW2.2, U1.3 (EN)
- net Reset: now also J9.2 (Pin_2)
- net Boot: now reaches SW3.2, U1.27 (IO0)
- net Boot: now also J9.3 (Pin_3)
- net vout renamed +5V
- net vout2 renamed +3V3
- net +3V3: now also J9.6 (Pin_6)
- new net: C15.1, IC1.6 (BAT), R16.2
- no-connect marks 4 -> 14
Other:
- note added: "Interfaces"
- note added: "Programming"
- moved on the sheet: C10, C11, C6, C7, D5, J5, J6, R1, R12, R13, R14, R2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
