File: _autosave-HaptiCare design.kicad_sch (KiCad schematic)
At the start: 60 parts, among them IC1 IP5306, J1 Conn_01x02_Socket, J2 Conn_01x02_Socket, J3 Conn_01x02_Socket, J4 Conn_01x02_Socket, J5 USB_C_Receptacle, J6 oled, J7 Conn_01x04_Pin, J8 Battery, Q1 AO3400A, Q2 AO3400A, Q3 AO3400A, Q4 AO3400A, SW1 SW_Push, SW2 SW_Push, SW3 SW_Push, U1 ESP32-S3-WROOM-1, U2 ME6211C33M5, U3 USBLC6-2P6

Commit message: add ESD protection
Parts:
- added R16: 10k, symbol Device:R_US
Connections:
- net vout2 is gone; now on net +3.3V: C10.1, C12.1, C13.1, J6.1 (Pin_1), J7.4 (Pin_4), R15.2, U1.2 (3V3), U2.5 (V_{OUT})
- net +3.3V: now also R16.2
- net GND: now also J6.4 (Pin_4); no longer J6.2 (Pin_2)
- net SCL: now also J6.3 (Pin_3); no longer J6.4 (Pin_4)
- net SDA: now also J6.2 (Pin_2); no longer J6.3 (Pin_3)
- net at SW3.2, U1.27 (IO0): now also R16.1
Other:
- moved on the sheet: SW3
